File: Witcher/LittleKiran.kicad_pcb (KiCad board)
At the start: 2 copper layers, 39 x 37 mm, 19 parts, among them J1 XT60PW-M, J2 XT60PW-M, J3 XT60PW-F, Q1 PXP012-30QLJ, Q2 PXP012-30QLJ, Q3 PXP012-30QLJ, Q4 FDN340P, U1 LTC4412xS6, U2 LTC4412xS6

Commit message: fixes
Parts:
- removed Q1: PXP012-30QLJ, iclr:PXP01230QLJ
- added Q5: SQS141ELNW-T1_GE3, iclr:SQS850ENT1_GE3, F.Cu at (138.3, 81.9)
- Q2, Q3: value PXP012-30QLJ -> SQS141ELNW-T1_GE3; footprint iclr:PXP01230QLJ -> iclr:SQS850ENT1_GE3
- moved Q4 25.9 mm to (140.9, 95.4), turned to 0 degrees
- moved D1 21.1 mm to (138.3, 95.2), turned to 90 degrees
- moved R3 20.0 mm to (139.7, 92.2), turned to -90 degrees
- moved R4 18.7 mm to (138.2, 92.2), turned to -90 degrees
- moved D2 15.4 mm to (146.0, 79.2), turned to 180 degrees
- moved R5 14.7 mm to (144.3, 77.7)
- moved Q2 3.70 mm to (138.3, 87.8)
- moved R2 3.69 mm to (129.6, 80.6)
- moved Q3 2.24 mm to (126.6, 88.1), turned to 180 degrees
- moved H1 1.51 mm to (144.2, 83.5)
- moved H3 1.50 mm to (115.0, 83.5)
- moved U1 1.21 mm to (132.0, 82.6), turned to -90 degrees
- moved U2 0.44 mm to (127.5, 83.8)
- moved R1 0.34 mm to (127.4, 81.4)
Connections:
- J3 pad 1: /SENSE -> GND
- J3 pad 2: GND -> /SENSE
- Q2 pad 5: Net-(J1-+) -> /SENSE
- Q2 pad 6: Net-(J1-+) -> /SENSE
- Q2 pad 7: Net-(J1-+) -> /SENSE
- Q2 pad 8: Net-(J1-+) -> /SENSE
- Q2 pad 9: Net-(J1-+) -> /SENSE
- Q3 pad 1: Net-(Q2-S_1) -> /SENSE
- Q3 pad 2: Net-(Q2-S_1) -> /SENSE
- Q3 pad 3: Net-(Q2-S_1) -> /SENSE
- Q3 pad 4: /GATE1 -> Net-(Q3-G)
- Q3 pad 5: /SENSE -> Net-(J2-+)
- Q3 pad 6: /SENSE -> Net-(J2-+)
- Q3 pad 7: /SENSE -> Net-(J2-+)
- Q3 pad 8: /SENSE -> Net-(J2-+)
- Q3 pad 9: /SENSE -> Net-(J2-+)
- R5 pad 1: Net-(Q2-S_1) -> Net-(J1-+)
- U2 pad 5: Net-(Q1-G) -> Net-(Q3-G)
Routing:
- net /GATE1: track 9.85 -> 17.5 mm
- net /SENSE: track 7.51 -> 0.00 mm, vias 21 -> 31
- net Net-(Q2-S_1): track 6.66 -> 0.00 mm, vias 8 -> 18
- net Net-(Q1-G): track 6.52 -> 0.00 mm
- net Net-(Q3-G): track 0.00 -> 4.19 mm
- net GND: track 0.00 -> 4.05 mm, vias 3 -> 28
- net Net-(U1-CTL): track 6.19 -> 2.90 mm
- net /STAT: track 19.8 -> 22.4 mm
- net Net-(J2-+): vias 20 -> 31
- net Net-(J1-+): vias 17 -> 26
