File: Witcher/LittleKiran.kicad_sch (KiCad schematic)
At the start: 17 parts, among them J1 XT60PW-M, J2 XT60PW-M, J3 XT60PW-M, Q1 PXP012-30QLJ, Q2 PXP012-30QLJ, Q3 PXP012-30QLJ, Q4 FDN340P, U1 LTC4412xS6, U2 LTC4412xS6

Commit message: kiran fixes
Parts:
- removed H2: MountingHole_Pad, MountingHole:MountingHole_3.2mm_M3_DIN965_Pad, symbol Mechanical:MountingHole_Pad
- removed J3: XT60PW-M, iclr:AMASS_XT60PW-M, symbol iclr:XT60PW-M
- added D2: BATT_LED, LED_SMD:LED_0603_1608Metric, symbol Device:LED
- added J3: XT60PW-F, iclr:AMASS_XT60PW-F, symbol iclr:XT60PW-F
- added R5: 3k, Resistor_SMD:R_0603_1608Metric, symbol Device:R_Small
Connections:
- net GND: now also D2.1 (K), J3.2
- net SENSE: now also J3.1
- net at Q2.1 (S_1), Q2.2 (S_2), Q2.3 (S_3)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: now also R5.1
- new net: J3.S1 (SHIELD), J3.S2 (SHIELD)
- new net: D2.2 (A), R5.2
- no-connect marks 1 -> 2
Changed lines of the file:
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@@
   (junction (at 187.452 38.1) (diameter 0) (color 0 0 0 0)
   )
+  (junction (at 159.258 38.1) (diameter 0) (color 0 0 0 0)
+  )
   (junction (at 129.54 43.18) (diameter 0) (color 0 0 0 0)
   )
@@
   )
   (no_connect (at 162.56 116.84))
+  (no_connect (at 203.2 99.06))
+  (wire (pts (xy 159.258 20.32) (xy 159.258 38.1))
+    (stroke (width 0) (type default))
+  )
   (wire (pts (xy 129.54 38.1) (xy 129.54 40.64))
     (stroke (width 0) (type default))
@@
     (stroke (width 0) (type default))
   )
-  (wire (pts (xy 154.94 38.1) (xy 162.052 38.1))
+  (wire (pts (xy 154.94 38.1) (xy 159.258 38.1))
     (stroke (width 0) (type default))
   )
@@
   )
   (wire (pts (xy 162.56 111.76) (xy 170.18 111.76))
+    (stroke (width 0) (type default))
+  )
+  (wire (pts (xy 159.258 38.1) (xy 162.052 38.1))
     (stroke (width 0) (type default))
   )
@@
     )
   )
+  (symbol (lib_name "GND_2") (lib_id "power:GND") (at 171.958 20.32 0) (unit 1)
+    (in_bom yes) (on_board yes) (dnp no) (fields_autoplaced)
+    (property "Reference" "#PWR03" (at 171.958 26.67 0)
+      (effects (font (size 1.27 1.27)) hide)
+    )
+    (property "Value" "GND" (at 171.958 24.4555 0)
+      (effects (font (size 1.27 1.27)))
+    )
+    (property "Footprint" "" (at 171.958 20.32 0)
+      (effects (font (size 1.27 1.27)) hide)
+    )
+    (property "Datasheet" "" (at 171.958 20.32 0)
+      (effects (font (size 1.27 1.27)) hide)
+    )
+    (pin "1")
+    (instances
+      (project "LittleKiran"
+        (path "/e63e39d7-6ac0-4ffd-8aa3-1841a4541b55"
+          (reference "#PWR03") (unit 1)
+        )
+      )
+    )
+  )
   (symbol (lib_id "power:GND") (at 101.6 137.16 0) (unit 1)
     (in_bom yes) (on_board yes) (dnp no) (fields_autoplaced)
@@
     )
   )
-  (symbol (lib_id "Mechanical:MountingHole_Pad") (at 150.876 175.26 0) (unit 1)
-    (in_bom yes) (on_board yes) (dnp no) (fields_autoplaced)
-    (property "Reference" "H2" (at 153.416 172.7199 0)
-      (effects (font (size 1.27 1.27)) (justify left))
-    )
-    (property "Value" "MountingHole_Pad" (at 153.416 175.2599 0)
-      (effects (font (size 1.27 1.27)) (justify left))
-    )
-    (property "Footprint" "MountingHole:MountingHole_3.2mm_M3_DIN965_Pad" (at 150.876 175.26 0)
-      (effects (font (size 1.27 1.27)) hide)
-    )
-    (property "Datasheet" "~" (at 150.876 175.26 0)
-      (effects (font (size 1.27 1.27)) hide)
-    )
-    (pin "1")
-    (instances
-      (project "LittleKiran"
-        (path "/e63e39d7-6ac0-4ffd-8aa3-1841a4541b55"
-          (reference "H2") (unit 1)
-        )
-      )
-    )
-  )
-  (symbol (lib_id "Mechanical:MountingHole_Pad") (at 140.716 175.26 0) (unit 1)
-    (in_bom yes) (on_board yes) (dnp no) (fields_autoplaced)
-    (property "Reference" "H1" (at 143.256 172.7199 0)
-      (effects (font (size 1.27 1.27)) (justify left))
-    )
-    (property "Value" "MountingHole_Pad" (at 143.256 175.2599 0)
-      (effects (font (size 1.27 1.27)) (justify left))
-    )
-    (property "Footprint" "MountingHole:MountingHole_3.2mm_M3_DIN965_Pad" (at 140.716 175.26 0)
-      (effects (font (size 1.27 1.27)) hide)
-    )
-    (property "Datasheet" "~" (at 140.716 175.26 0)
-      (effects (font (size 1.27 1.27)) hide)
-    )
-    (pin "1")
-    (instances
-      (project "LittleKiran"
-        (path "/e63e39d7-6ac0-4ffd-8aa3-1841a4541b55"
-          (reference "H1") (unit 1)
-        )
-      )
-    )
-  )
-  (symbol (lib_id "power:GND") (at 149.86 81.28 0) (unit 1)
-    (in_bom yes) (on_board yes) (dnp no) (fields_autoplaced)
-    (property "Reference" "#PWR0102" (at 149.86 87.63 0)
-      (effects (font (size 1.27 1.27)) hide)
-    )
-    (property "Value" "GND" (at 149.86 85.7234 0)
-      (effects (font (size 1.27 1.27)))
-    )
-    (property "Footprint" "" (at 149.86 81.28 0)
-      (effects (font (size 1.27 1.27)) hide)
-    )
-    (property "Datasheet" "" (at 149.86 81.28 0)
-      (effects (font (size 1.27 1.27)) hide)
-    )
-    (pin "1")
-    (instances
-      (project "LittleKiran"
-        (path "/e63e39d7-6ac0-4ffd-8aa3-1841a4541b55"
-          (reference "#PWR0102") (unit 1)
-        )
-      )
-    )
-  )
-  (symbol (lib_id "iclr:XT60PW-M") (at 213.36 93.98 0) (unit 1)
-    (in_bom yes) (on_board yes) (dnp no) (fields_autoplaced)
-    (property "Reference" "J3" (at 219.202 91.8753 0)
-      (effects (font (size 1.27 1.27)) (justify left))
-    )
-    (property "Value" "XT60PW-M" (at 219.202 94.4122 0)
-      (effects (font (size 1.27 1.27)) (justify left))
-    )
-    (property "Footprint" "iclr:AMASS_XT60PW-M" (at 213.36 93.98 0)
+  (symbol (lib_id "iclr:XT60PW-F") (at 213.36 93.98 0) (unit 1)
+    (in_bom yes) (on_board yes) (dnp no) (fields_autoplaced)
+    (property "Reference" "J3" (at 219.202 94.6063 0)
+      (effects (font (size 1.27 1.27)) (justify left))
+    )
+    (property "Value" "XT60PW-F" (at 219.202 96.5273 0)
+      (effects (font (size 1.27 1.27)) (justify left))
+    )
+    (property "Footprint" "iclr:AMASS_XT60PW-F" (at 213.36 93.98 0)
       (effects (font (size 1.27 1.27)) (justify bottom) hide)
     )
@@
       (effects (font (size 1.27 1.27)) hide)
     )
-    (property "STANDARD" "Manufacturer recommendations" (at 213.36 93.98 0)
+    (property "PARTREV" "V1.2" (at 213.36 93.98 0)
+      (effects (font (size 1.27 1.27)) (justify bottom) hide)
+    )
+    (property "STANDARD" "Manufacturer Recommendations" (at 213.36 93.98 0)
+      (effects (font (size 1.27 1.27)) (justify bottom) hide)
+    )
+    (property "MAXIMUM_PACKAGE_HEIGHT" "8.4 mm" (at 213.36 93.98 0)
       (effects (font (size 1.27 1.27)) (justify bottom) hide)
     )
@@
       (effects (font (size 1.27 1.27)) (justify bottom) hide)
     )
-    (property "PARTREV" "V1.2" (at 213.36 93.98 0)
-      (effects (font (size 1.27 1.27)) (justify bottom) hide)
-    )
-    (property "MAXIMUM_PACKAGE_HEIGHT" "8.4 mm" (at 213.36 93.98 0)
-      (effects (font (size 1.27 1.27)) (justify bottom) hide)
-    )
-    (pin "1")
-    (pin "2")
+    (pin "1")
+    (pin "2")
+    (pin "S1")
+    (pin "S2")
     (instances
       (project "LittleKiran"
         (path "/e63e39d7-6ac0-4ffd-8aa3-1841a4541b55"
           (reference "J3") (unit 1)
+        )
+      )
+    )
+  )
+  (symbol (lib_id "Mechanical:MountingHole_Pad") (at 140.716 175.26 0) (unit 1)
+    (in_bom yes) (on_board yes) (dnp no) (fields_autoplaced)
+    (property "Reference" "H1" (at 143.256 172.7199 0)
+      (effects (font (size 1.27 1.27)) (justify left))
+    )
+    (property "Value" "MountingHole_Pad" (at 143.256 175.2599 0)
+      (effects (font (size 1.27 1.27)) (justify left))
+    )
+    (property "Footprint" "MountingHole:MountingHole_3.2mm_M3_DIN965_Pad" (at 140.716 175.26 0)
+      (effects (font (size 1.27 1.27)) hide)
+    )
+    (property "Datasheet" "~" (at 140.716 175.26 0)
+      (effects (font (size 1.27 1.27)) hide)
+    )
+    (pin "1")
+    (instances
+      (project "LittleKiran"
+        (path "/e63e39d7-6ac0-4ffd-8aa3-1841a4541b55"
+          (reference "H1") (unit 1)
+        )
+      )
+    )
+  )
+  (symbol (lib_id "power:GND") (at 149.86 81.28 0) (unit 1)
+    (in_bom yes) (on_board yes) (dnp no) (fields_autoplaced)
+    (property "Reference" "#PWR0102" (at 149.86 87.63 0)
+      (effects (font (size 1.27 1.27)) hide)
+    )
+    (property "Value" "GND" (at 149.86 85.7234 0)
+      (effects (font (size 1.27 1.27)))
+    )
+    (property "Footprint" "" (at 149.86 81.28 0)
+      (effects (font (size 1.27 1.27)) hide)
+    )
+    (property "Datasheet" "" (at 149.86 81.28 0)
+      (effects (font (size 1.27 1.27)) hide)
+    )
+    (pin "1")
+    (instances
+      (project "LittleKiran"
+        (path "/e63e39d7-6ac0-4ffd-8aa3-1841a4541b55"
+          (reference "#PWR0102") (unit 1)
         )
       )
@@
         )
       )
+    )
+  )
+  (symbol (lib_id "Device:R_Small") (at 161.798 20.32 90) (unit 1)
+    (in_bom yes) (on_board yes) (dnp no) (fields_autoplaced)
+    (property "Reference" "R5" (at 161.798 16.5735 90)
+      (effects (font (size 1.27 1.27)))
+    )
+    (property "Value" "3k" (at 161.798 18.4945 90)
+      (effects (font (size 1.27 1.27)))
+    )
+    (property "Footprint" "Resistor_SMD:R_0603_1608Metric" (at 161.798 20.32 0)
+      (effects (font (size 1.27 1.27)) hide)
+    )
+    (property "Datasheet" "~" (at 161.798 20.32 0)
+      (effects (font (size 1.27 1.27)) hide)
+    )
+    (pin "1")
+    (pin "2")
+    (instances
+      (project "LittleKiran"
+        (path "/e63e39d7-6ac0-4ffd-8aa3-1841a4541b55"
+          (reference "R5") (unit 1)
+        )
+      )
+    )
+  )
+  (symbol (lib_id "Device:LED") (at 168.148 20.32 180) (unit 1)
+    (in_bom yes) (on_board yes) (dnp no) (fields_autoplaced)
+    (property "Reference" "D2" (at 169.7355 15.1511 0)
+      (effects (font (size 1.27 1.27)))
+    )
+    (property "Value" "BATT_LED" (at 169.7355 17.0721 0)
+      (effects (font (size 1.27 1.27)))
+    )
+    (property "Footprint" "LED_SMD:LED_0603_1608Metric" (at 168.148 20.32 0)
+      (effects (font (size 1.27 1.27)) hide)
+    )
+    (property "Datasheet" "~" (at 168.148 20.32 0)
+      (effects (font (size 1.27 1.27)) hide)
+    )
+    (pin "1")
+    (pin "2")
+    (instances
+      (project "LittleKiran"
+        (path "/e63e39d7-6ac0-4ffd-8aa3-1841a4541b55"
+          (reference "D2") (unit 1)
+        )
+      )

Commit message: fixes
Parts:
- removed Q1, Q2, Q3: PXP012-30QLJ, iclr:PXP01230QLJ, symbol iclr:PXP012-30QLJ
- added Q2, Q3, Q5: SQS141ELNW-T1_GE3, SQS850ENT1_GE3, symbol iclr:SQS141ELNW-T1_GE3
Connections:
- net GATE1: now also Q2.4 (G), Q5.4 (G)
- net GND: now also J3.1; no longer J3.2
- net SENSE: now also J3.2, Q2.10 (D_6), Q2.11 (D_7), Q2.5 (D_1), Q2.6 (D_2), Q2.7 (D_3), Q2.8 (D_4), Q2.9 (D_5), Q3.1 (S_1), Q3.2 (S_2), Q3.3 (S_3); no longer J3.1
- net at J2.1 (+), R1.2, U2.1 (VIN): now also Q3.10 (D_6), Q3.11 (D_7), Q3.5 (D_1), Q3.6 (D_2), Q3.7 (D_3), Q3.8 (D_4), Q3.9 (D_5)
- net at U2.5 (GATE): now also Q3.4 (G)
- net at R5.1: now also J1.1 (+), U1.1 (VIN), Q5.10 (D_6), Q5.11 (D_7), Q5.5 (D_1), Q5.6 (D_2), Q5.7 (D_3), Q5.8 (D_4), Q5.9 (D_5)
- new net: Q2.1 (S_1), Q2.2 (S_2), Q2.3 (S_3), Q5.1 (S_1), Q5.2 (S_2), Q5.3 (S_3)
Other:
- moved on the sheet: D2, J3, R5

Commit message: v2.0
Parts:
- removed Q5: SQS141ELNW-T1_GE3, SQS850ENT1_GE3, symbol iclr:SQS141ELNW-T1_GE3
- added J4: Conn_01x02_Pin, Connector_Molex:Molex_Nano-Fit_105313-xx02_1x02_P2.50mm_Horizontal, symbol Connector:Conn_01x02_Pin
- added Q2, Q3: SQS141ELNW-T1_GE3, iclr:SQS850ENT1_GE3, symbol iclr:SQS141ELNW-T1_GE3
- added R3, R4, R5: 10k, Resistor_SMD:R_0402_1005Metric, symbol Device:R_Small
- Q1: renamed from Q3; footprint SQS850ENT1_GE3 -> iclr:SQS850ENT1_GE3
- Q4: renamed from Q2; footprint SQS850ENT1_GE3 -> iclr:SQS850ENT1_GE3
- R1: value 0 -> 470k; footprint Resistor_SMD:R_0603_1608Metric -> Resistor_SMD:R_0402_1005Metric
- R2: footprint Resistor_SMD:R_0603_1608Metric -> Resistor_SMD:R_0402_1005Metric
- renumbered Q4 to Q5, R5 to R6, R4 to R7, R3 to R8
Connections:
- net GATE1: now also Q3.4
- net GND: now also J4.2 (Pin_2), R5.2; no longer U2.3 (CTL)
- net VADP: now reaches J2.1 (+), Q1.10, Q1.11, Q1.5, Q1.6, Q1.7, Q1.8, Q1.9, R1.2, U2.1 (VIN)
- net GATE2: now reaches Q1.4, U2.5 (GATE)
- net GATE2: now also Q2.4
- net VBAT: now reaches J1.1 (+), R6.1, U1.1 (VIN)
- net VBAT: now also Q3.10, Q3.11, Q3.5, Q3.6, Q3.7, Q3.8, Q3.9
- net at R1.1, R2.1, U1.3 (CTL): now also R3.2
- net at Q4.1, Q4.2, Q4.3: now also Q3.1, Q3.2, Q3.3
- net SENSE renamed VOUT
- net VOUT: now also Q2.10, Q2.11, Q2.5, Q2.6, Q2.7, Q2.8, Q2.9; no longer Q1.1 (S_1), Q1.2 (S_2), Q1.3 (S_3)
- new net: R4.2, R5.1, U2.3 (CTL)
- new net: Q1.1, Q1.2, Q1.3, Q2.1, Q2.2, Q2.3
- new net VRST: J4.1 (Pin_1), R3.1, R4.1
Other:
- moved on the sheet: D1, D2, H1, H3, J1, J2, J3, Q5, R1, R2, R6, R7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

Commit message: my nanofit 3d model reset itself
Parts:
- J4: footprint Connector_Molex:Molex_Nano-Fit_105313-xx02_1x02_P2.50mm_Horizontal -> iclr:Molex_Nano-Fit_105313-xx02_1x02_P2.50mm_Horizontal
Changed lines of the file:
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@@
 			)
 		)
-		(property "Footprint" "Connector_Molex:Molex_Nano-Fit_105313-xx02_1x02_P2.50mm_Horizontal"
+		(property "Footprint" "iclr:Molex_Nano-Fit_105313-xx02_1x02_P2.50mm_Horizontal"
 			(at 60.96 91.44 0)
 			(effects

Commit message: Simulation model
Parts:
- R3, R4: value 10k -> 1k
Changed lines of the file:
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@@
 			)
 		)
-		(property "Value" "10k"
+		(property "Value" "1k"
 			(at 106.68 118.11 0)
 			(effects
@@
 			)
 		)
-		(property "Value" "10k"
+		(property "Value" "1k"
 			(at 80.772 67.31 0)
 			(effects
