File: Witcher/Witcher.kicad_sch (KiCad schematic)
At the start: 23 parts, among them J1 XT60PW-M, J2 XT60PW-M, J3 XT60PW-F, J4 Conn_01x02_Pin, Q1 SQS141ELNW-T1_GE3, Q2 SQS141ELNW-T1_GE3, Q3 SQS141ELNW-T1_GE3, Q4 SQS141ELNW-T1_GE3, Q5 FDN340P, U1 LTC4412xS6, U2 LTC4412xS6

Commit message: cleaned schematic and bom
Parts:
- D101: renamed from D2; value BATT_LED -> LED_YELLOW
- D102: renamed from D1; value SYS_LED -> LED_BLUE
- H101: renamed from H1; now left out of the parts list
- H102: renamed from H3; now left out of the parts list
- R101: renamed from R3; value 1k -> 1kΩ
- R102: renamed from R1; value 470k -> 470kΩ
- R103: renamed from R2; value 10k -> 10kΩ
- R104: renamed from R6; value 3k -> 3kΩ
- R105: renamed from R4; value 1k -> 1kΩ
- R106: renamed from R5; value 10k -> 10kΩ
- R107: renamed from R7; value 3k -> 3kΩ
- R108: renamed from R8; value 470k -> 470kΩ
- renumbered J4 to J101, J1 to J102, J2 to J103, J3 to J104, Q3 to Q101, Q1 to Q102, Q4 to Q103, Q2 to Q104, Q5 to Q105, U1 to U101, U2 to U102
